File: USB-C_PD_Board_V2_CYPD3177.kicad_sch (KiCad schematic)
At the start: 43 parts, among them J2 Type-C_6P, J3 I2C, J4 Conn_01x03, Q1 DMP3098LSD, SW3 SW_SPDT, SW4 SW_SPDT, U1 CYPD3177-24LQ

Commit message: layout started
Parts:
- removed JP1: SolderJumper_2_Open, Jumper:SolderJumper-2_P1.3mm_Open_RoundedPad1.0x1.5mm, symbol Jumper:SolderJumper_2_Open
- added D6: D_Zener, Diode_THT:D_DO-35_SOD27_P7.62mm_Horizontal, symbol Device:D_Zener
- J2: footprint Connector_USB:USB_C_Receptacle_GCT_USB4125-xx-x-0190_6P_TopMnt_Horizontal -> Custom:USB-C 6 Pin - Long pads
- SW3, SW4: footprint (none) -> SS12D00_switch:Schiebeschalter SS-12D00
Connections:
- net GND: now also J4.1 (Pin_1), J4.2 (Pin_2), J4.3 (Pin_3)
- net at Q1.1 (S), Q1.3 (S), R8.1: now also D6.1 (K)
- net at C4.2, C5.2, Q1.2 (G)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: now also D6.2 (A)
- no-connect marks 4 -> 5
Other:
- company: (none) -> Potpurri
- title: (none) -> USB-C Power Delivery Board
- moved on the sheet: D7, R8

Commit message: started routing
Parts:
- added H1, H2: MountingHole, MountingHole:MountingHole_3.2mm_M3_DIN965_Pad, symbol Mechanical:MountingHole
Connections:
- net VDD is gone; now on net +3V3: R11.1, R12.1
- net at R16.2, SW4.2 (B): now also U1.5 (ISNK_COARSE); no longer U1.2 (VBUS_MAX)
- net at R13.2, SW3.2 (B): now also U1.2 (VBUS_MAX); no longer U1.5 (ISNK_COARSE)
- net at R23.1: now also SW2.2; no longer SW2.1
- net at R22.1: now also SW2.5; no longer SW2.2
- net at SW2.3, SW2.4: now also SW4.3 (C); no longer SW4.1 (A)
- net at R21.1: now also SW2.6; no longer SW2.5
- net at R24.1: now also SW2.1; no longer SW4.3 (C)
Other:
- moved on the sheet: R17

Commit message: added turn on/off switch, added diode to indicate on state
Parts:
- removed J3: I2C, Connector_PinHeader_2.54mm:PinHeader_1x02_P2.54mm_Vertical, symbol Connector_Generic:Conn_01x02
- added D7: LED, LED_SMD:LED_0805_2012Metric, symbol Device:LED
- added R10: 1k, Resistor_SMD:R_0603_1608Metric, symbol Device:R
- added SW3: SW_SPDT, SS12D00_switch:Schiebeschalter SS-12D00, symbol Switch:SW_SPDT
- added TP3 (x2): TestPoint, TestPoint:TestPoint_Pad_1.0x1.0mm, symbol Connector:TestPoint
Connections:
- net GND: now also D7.1 (K)
- net VBUS: now also R10.2, SW3.2 (B), SW3.3 (C); no longer J2.A9 (VBUS), J2.B9 (VBUS)
- net at R12.2, U1.12 (HPI_SDA): now also TP3.1
- net at R11.2, U1.13 (HPI_SCL): now also TP3.1
- new net: D7.2 (A), R10.1
- new net: J2.A9 (VBUS), J2.B9 (VBUS), SW3.1 (A)
Other:
- moved on the sheet: C1, J2
